Commit message: Actualizacion de archivos

File: description/lidar.xacro (robot description, xacro)
@@ -4,10 +4,10 @@
         <parent link="chassis"/>
         <child link="laser_frame"/>
-        <origin xyz="0.1 0 0.175" rpy="0 0 0"/>
+        <origin xyz="0.18 0 0.140" rpy="0 0 0"/>
     </joint>
     <link name="laser_frame">
         <visual>
             <geometry>
-                <cylinder radius="0.05" length="0.04"/>
+                <cylinder radius="0.018" length="0.035"/>
             </geometry>
             <material name="red"/>
@@ -15,8 +15,8 @@
         <collision>
             <geometry>
-                <cylinder radius="0.05" length="0.04"/>
+                <cylinder radius="0.018" length="0.035"/>
             </geometry>
         </collision>
-        <xacro:inertial_cylinder mass="0.1" length="0.04" radius="0.05">
+        <xacro:inertial_cylinder mass="0.1" length="0.035" radius="0.02">
             <origin xyz="0 0 0" rpy="0 0 0"/>
         </xacro:inertial_cylinder>
@@ -26,5 +26,5 @@
         <sensor name="laser" type="ray">
             <pose> 0 0 0 0 0 0 </pose>
-            <visualize>true</visualize>
+            <visualize>false</visualize>
             <update_rate>10</update_rate>
             <ray>

File: description/robot.urdf.xacro (robot description, xacro)
@@ -2,5 +2,7 @@
 <robot xmlns:xacro="http://www.ros.org/wiki/xacro"  name="robot">
     <xacro:include filename="robot_core.xacro" />
-    <xacro:include filename="gazebo_control.xacro" />
+    <!-- <xacro:include filename="gazebo_control.xacro" /> -->
+    <xacro:include filename="ros2_control.xacro" />
     <xacro:include filename="lidar.xacro" />
+    <xacro:include filename="camera.xacro" />
 </robot>

File: description/robot_core.xacro (robot description, xacro)
@@ -24,22 +24,23 @@
         <parent link="base_link"/>
         <child link="chassis"/>
-        <origin xyz="-0.1 0 0"/>
+        <!--<origin xyz="-0.1 0 1.5708"/>-->
+        <origin xyz="0 0 0"/>
     </joint>
     <link name="chassis">
         <visual>
-            <origin xyz="0.15 0 0.075"/>
+            <origin xyz="0.144 0 0.061"/>  <!-- se desplaza xyz= x/2 0 z/2 para no estar en el centro del grid, a z sumar el radio de la rueda -->
             <geometry>
-                <box size="0.3 0.3 0.15"/>
+                <box size="0.288 0.16 0.122"/> <!-- Dimensiones del cuerpo -->
             </geometry>
             <material name="white"/>
         </visual>
         <collision>
-            <origin xyz="0.15 0 0.075"/>
+            <origin xyz="0.144 0 0.061"/>
             <geometry>
-                <box size="0.3 0.3 0.15"/>
+                <box size="0.288 0.16 0.122"/>
             </geometry>
         </collision>
-        <xacro:inertial_box mass="0.5" x="0.3" y="0.3" z="0.3">
-            <origin xyz="0.15 0 0.075" rpy="0 0 0"/>
+        <xacro:inertial_box mass="2" x="0.288" y="0.16" z="0.122">
+            <origin xyz="0.144 0 0.061" rpy="0 0 0"/>
         </xacro:inertial_box>
     </link>
@@ -51,5 +52,5 @@
         <parent link="base_link"/>
         <child link="left_wheel"/>
-        <origin xyz="0 0.175 0" rpy="-${pi/2} 0 0"/>
+        <origin xyz="0.072 0.093 0" rpy="-${pi/2} 0 0"/> <!-- A 9.3 cm en y del base_link, y rotado a 90 en x -->
         <axis xyz="0 0 1"/>
     </joint>
@@ -57,5 +58,5 @@
         <visual>
             <geometry>
-                <cylinder length="0.04" radius="0.05" />
+                <cylinder length="0.026" radius="0.0335" />
             </geometry>
             <material name="blue"/>
@@ -63,8 +64,8 @@
         <collision>
             <geometry>
-                <cylinder length="0.04" radius="0.05" />
+                <cylinder length="0.026" radius="0.0335" />
             </geometry>
         </collision>
-        <xacro:inertial_cylinder mass="0.1" length="0.04" radius="0.05">
+        <xacro:inertial_cylinder mass="0.1" length="0.026" radius="0.0335">
             <origin xyz="0 0 0" rpy="0 0 0"/>
         </xacro:inertial_cylinder>
@@ -77,5 +78,5 @@
         <parent link="base_link"/>
         <child link="right_wheel"/>
-        <origin xyz="0 -0.175 0" rpy="${pi/2} 0 0"/>
+        <origin xyz="0.072 -0.093 0" rpy="${pi/2} 0 0"/>
         <axis xyz="0 0 -1"/>
     </joint>
@@ -83,5 +84,5 @@
         <visual>
             <geometry>
-                <cylinder length="0.04" radius="0.05" />
+                <cylinder length="0.026" radius="0.0335" />
             </geometry>
             <material name="blue"/>
@@ -89,8 +90,8 @@
         <collision>
             <geometry>
-                <cylinder length="0.04" radius="0.05" />
+                <cylinder length="0.026" radius="0.0335" />
             </geometry>
         </collision>
-        <xacro:inertial_cylinder mass="0.1" length="0.04" radius="0.05">
+        <xacro:inertial_cylinder mass="0.1" length="0.026" radius="0.0335">
             <origin xyz="0 0 0" rpy="0 0 0"/>
         </xacro:inertial_cylinder>
@@ -108,5 +109,5 @@
         <visual>
             <geometry>
-                <sphere radius="0.05" />
+                <sphere radius="0.03" />
             </geometry>
             <material name="black"/>
@@ -114,8 +115,8 @@
         <collision>
             <geometry>
-                <sphere radius="0.05" />
+                <sphere radius="0.03" />
             </geometry>
         </collision>
-        <xacro:inertial_sphere mass="0.01" radius="0.05">
+        <xacro:inertial_sphere mass="0.01" radius="0.03">
             <origin xyz="0 0 0" rpy="0 0 0"/>
         </xacro:inertial_sphere>
